File: k22-brd/k22-brd.brd (EAGLE design)
At the start: 25.4 x 80 mm, 34 parts, among them IC1 LMS8117, J1 61302011121, J2 61302011121, J3 CORTEX_DEBUG_PTH

Commit message: Basic routing done
Parts:
- removed IC1: LMS8117, IC_Power-Management:SOT230P700X170-4
- added U$2: LMS8117AMP-3.3, vym0038_k22_misc:SOT223
- U$4: value USBLC6-2SC6 -> USBLC6-4SC6Y
- moved LED_PTD5 86.6 mm to (16.3, 46.3), turned to 270 degrees
- moved J3 76.6 mm to (11.6, 7.86)
- moved CV2 75.9 mm to (14.6, 43.5), flipped to the bottom, turned to 180 degrees
- moved RU2 73.4 mm to (10.2, 59.9), flipped to the bottom, turned to 90 degrees
- moved RU1 69.6 mm to (12.7, 59.9), flipped to the bottom, turned to 90 degrees
- moved DV1 69.6 mm to (8.48, 51.3), flipped to the bottom, turned to 90 degrees
- moved CV1 68.2 mm to (12.3, 53.4), flipped to the bottom, turned to 180 degrees
- moved SJS2 64.2 mm to (6.27, 14.7), turned to 90 degrees
- moved SJS1 62.4 mm to (8.57, 14.7), turned to 90 degrees
- moved SJM2 62.0 mm to (13.1, 14.7), turned to 270 degrees
- moved CM3 60.3 mm to (11.8, 21.0), flipped to the bottom
- moved CM4 59.7 mm to (10.5, 30.8), flipped to the bottom
- moved RR1 58.9 mm to (6.15, 35.7), flipped to the bottom
- moved SJM1 57.5 mm to (10.8, 14.7), turned to 270 degrees
- moved CM2 54.9 mm to (11.8, 23.1), flipped to the bottom
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Connections:
- removed net V3V: CM1.2, CM2.2, CM3.2
- new net N$5: J1.4
- net 3V3: now also CM1.2, CM2.2, CM3.2, J1.5, U$2.2, U$2.4; no longer IC1.2
- net D+CON: no longer U$4.6
- net D-CON: no longer U$4.4
- net DM0: now also J1.9
- net DP0: now also J1.8
- net GND: now also J1.1, J1.10, J1.6, U$2.1; no longer IC1.1, IC1.4
- net PTD4: now also SWB.3; no longer SWB.1
- net RESET: now also J1.7
- net SWD_CLK: now also J1.12
- net SWD_DIO: now also J1.15
- net UART_RX: now also J1.14
- net UART_TX: now also J1.13
- net USB5V: now also J1.3
- net VI: now also U$2.3; no longer IC1.3
- net VIN: now also J1.2
- net VREF: now also J1.11
Routing:
- net 3V3: track 0.00 -> 90.4 mm, vias 0 -> 6
- net USB5V: track 0.00 -> 45.7 mm, vias 0 -> 2
- net RESET: track 0.00 -> 37.8 mm, vias 0 -> 1
- net PTB1: track 0.00 -> 33.5 mm
- net PTB0: track 0.00 -> 31.2 mm
- net PTD7: track 0.00 -> 26.8 mm
- net PTD6: track 0.00 -> 25.0 mm
- net PTD5: track 0.00 -> 24.5 mm
- net SWD_CLK: track 0.00 -> 24.4 mm, vias 0 -> 1
- net PTB2: track 0.00 -> 22.6 mm
- net SWD_DIO: track 0.00 -> 21.3 mm, vias 0 -> 1
- net USBGNDSHIELD: track 0.00 -> 20.3 mm
- net PTB3: track 0.00 -> 20.2 mm
- net D-CON: track 0.00 -> 20.1 mm
- net D+CON: track 0.00 -> 19.6 mm
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- added copper zone on layer 1, net GND
- added copper zone on layer 16, net GND
- added copper zone on layer 1, net GNDCUTOU
- added copper zone on layer 16, net GNDCUTOU
Other:
- board size 25.4 x 80 mm -> 22.9 x 63.5 mm

Commit message: Fixed routing
Routing:
- net 3V3: track 90.4 -> 91.7 mm
- net VBUSCON: track 12.1 -> 13.1 mm
- net D+CON: track 19.6 -> 19.0 mm
- net GND: vias 34 -> 35
