File: opensda-shield/opensda-shield.brd (EAGLE design)
At the start: 21.6 x 53.3 mm, 17 parts, among them IC1 74LVC125, IC2 74LVC125, J1 61302011121, J2 61302011121, J3 61300211121, J4 CORTEX_DEBUG_PTH, J5 61301511121

Commit message: drobne upravy
Parts:
- moved R6 1.27 mm to (6.99, 14.0)
- moved J4 0.95 mm to (10.8, 9.21)
- moved LED1 0.95 mm to (6.03, 49.5)
- moved C2 0.32 mm to (11.1, 20.0)
- moved R5 0.32 mm to (8.57, 49.5)
Routing:
- net 3V3: track 81.1 -> 79.5 mm
- net !RST_TGT: track 37.3 -> 36.3 mm
- net N$2: track 2.01 -> 2.64 mm
- net SWD_CLK_TGT: track 33.5 -> 32.9 mm
- net SWD_DIO_TGT: track 52.4 -> 51.8 mm
